File: hardware/ESC.kicad_sch (KiCad schematic)
At the start: 91 parts, among them J1 +, J10 +, J2 -, J3 +, J4 +, J5 +, J6 +, J7 Conn_01x03, J8 +, J9 +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

Commit message: updated production files
Parts:
- L1: value 27uH -> 33uH
- Q7: value AGM60P30A -> AGM60P30AP
Other:
- moved on the sheet: C24, C33, Y1
Changed lines of the file:
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@@
 	)
 	(junction
-		(at 148.59 92.71)
+		(at 149.86 92.71)
 		(diameter 0)
 		(color 0 0 0 0)
@@
 	)
 	(junction
-		(at 165.1 92.71)
+		(at 166.37 92.71)
 		(diameter 0)
 		(color 0 0 0 0)
@@
 	(wire
 		(pts
-			(xy 165.1 101.6) (xy 165.1 102.87)
+			(xy 166.37 101.6) (xy 166.37 102.87)
 		)
 		(stroke
@@
 	(wire
 		(pts
-			(xy 161.29 92.71) (xy 165.1 92.71)
+			(xy 162.56 92.71) (xy 166.37 92.71)
 		)
 		(stroke
@@
 	(wire
 		(pts
-			(xy 148.59 92.71) (xy 148.59 93.98)
+			(xy 149.86 92.71) (xy 149.86 93.98)
 		)
 		(stroke
@@
 	(wire
 		(pts
-			(xy 157.48 85.09) (xy 151.13 85.09)
+			(xy 158.75 85.09) (xy 152.4 85.09)
 		)
 		(stroke
@@
 	(wire
 		(pts
-			(xy 157.48 87.63) (xy 157.48 85.09)
+			(xy 158.75 87.63) (xy 158.75 85.09)
 		)
 		(stroke
@@
 	(wire
 		(pts
-			(xy 165.1 92.71) (xy 165.1 93.98)
+			(xy 166.37 92.71) (xy 166.37 93.98)
 		)
 		(stroke
@@
 	(wire
 		(pts
-			(xy 148.59 101.6) (xy 148.59 102.87)
+			(xy 149.86 101.6) (xy 149.86 102.87)
 		)
 		(stroke
@@
 	(wire
 		(pts
-			(xy 153.67 92.71) (xy 148.59 92.71)
+			(xy 154.94 92.71) (xy 149.86 92.71)
 		)
 		(stroke
@@
 	(wire
 		(pts
-			(xy 151.13 85.09) (xy 151.13 86.36)
+			(xy 152.4 85.09) (xy 152.4 86.36)
 		)
 		(stroke
@@
 	(wire
 		(pts
-			(xy 142.24 92.71) (xy 148.59 92.71)
+			(xy 143.51 92.71) (xy 149.86 92.71)
 		)
 		(stroke
@@
 	(wire
 		(pts
-			(xy 157.48 97.79) (xy 157.48 99.06)
+			(xy 158.75 97.79) (xy 158.75 99.06)
 		)
 		(stroke
@@
 	(wire
 		(pts
-			(xy 165.1 92.71) (xy 173.99 92.71)
+			(xy 166.37 92.71) (xy 175.26 92.71)
 		)
 		(stroke
@@
 	)
 	(label "HSE_IN"
-		(at 142.24 92.71 0)
+		(at 143.51 92.71 0)
 		(effects
 			(font
@@
 	)
 	(label "HSE_OUT"
-		(at 173.99 92.71 180)
+		(at 175.26 92.71 180)
 		(effects
 			(font
@@
 	(symbol
 		(lib_id "Device:C")
-		(at 165.1 97.79 0)
+		(at 166.37 97.79 0)
 		(unit 1)
 		(body_style 1)
@@
 		(dnp no)
 		(property "Reference" "C33"
-			(at 166.116 95.504 0)
+			(at 167.386 95.504 0)
 			(show_name no)
 			(do_not_autoplace no)
@@
 		)
 		(property "Value" "8.2pF"
-			(at 166.37 100.33 0)
+			(at 167.64 100.33 0)
 			(show_name no)
 			(do_not_autoplace no)
@@
 		)
 		(property "Footprint" "Capacitor_SMD:C_0402_1005Metric"
-			(at 166.0652 101.6 0)
+			(at 167.3352 101.6 0)
 			(hide yes)
 			(show_name no)
@@
 		)
 		(property "Datasheet" ""
-			(at 165.1 97.79 0)
+			(at 166.37 97.79 0)
 			(hide yes)
 			(show_name no)
@@
 		)
 		(property "Description" "Unpolarized capacitor"
-			(at 165.1 97.79 0)
+			(at 166.37 97.79 0)
 			(hide yes)
 			(show_name no)
@@
 	(symbol
 		(lib_id "power:GND")
-		(at 151.13 86.36 0)
+		(at 152.4 86.36 0)
 		(unit 1)
 		(body_style 1)
@@
 		(dnp no)
 		(property "Reference" "#PWR051"
-			(at 151.13 92.71 0)
+			(at 152.4 92.71 0)
 			(hide yes)
 			(show_name no)
@@
 		)
 		(property "Value" "GND"
-			(at 151.13 90.17 0)
+			(at 152.4 90.17 0)
 			(show_name no)
 			(do_not_autoplace no)
@@
 		)
 		(property "Footprint" ""
-			(at 151.13 86.36 0)
+			(at 152.4 86.36 0)
 			(hide yes)
 			(show_name no)
@@
 		)
 		(property "Datasheet" ""
-			(at 151.13 86.36 0)
+			(at 152.4 86.36 0)
 			(hide yes)
 			(show_name no)
@@
 		)
 		(property "Description" "Power symbol creates a global label with name \"GND\" , ground"
-			(at 151.13 86.36 0)
+			(at 152.4 86.36 0)
 			(hide yes)
 			(show_name no)
@@
 	(symbol
 		(lib_id "power:GND")
-		(at 157.48 99.06 0)
+		(at 158.75 99.06 0)
 		(unit 1)
 		(body_style 1)
@@
 		(dnp no)
 		(property "Reference" "#PWR050"
-			(at 157.48 105.41 0)
+			(at 158.75 105.41 0)
 			(hide yes)
 			(show_name no)
@@
 		)
 		(property "Value" "GND"
-			(at 157.48 102.87 0)
+			(at 158.75 102.87 0)
 			(show_name no)
 			(do_not_autoplace no)
@@
 		)
 		(property "Footprint" ""
-			(at 157.48 99.06 0)
+			(at 158.75 99.06 0)
 			(hide yes)
 			(show_name no)
@@
 		)
 		(property "Datasheet" ""
-			(at 157.48 99.06 0)
+			(at 158.75 99.06 0)
 			(hide yes)
 			(show_name no)
@@
 		)
 		(property "Description" "Power symbol creates a global label with name \"GND\" , ground"
-			(at 157.48 99.06 0)
+			(at 158.75 99.06 0)
 			(hide yes)
 			(show_name no)
@@
 	(symbol
 		(lib_id "power:GND")
-		(at 165.1 102.87 0)
+		(at 166.37 102.87 0)
 		(unit 1)
 		(body_style 1)
@@
 		(dnp no)
 		(property "Reference" "#PWR049"
-			(at 165.1 109.22 0)
+			(at 166.37 109.22 0)
 			(hide yes)
 			(show_name no)
@@
 		)
 		(property "Value" "GND"
-			(at 165.1 106.68 0)
+			(at 166.37 106.68 0)
 			(show_name no)
 			(do_not_autoplace no)
@@
 		)
 		(property "Footprint" ""
-			(at 165.1 102.87 0)
+			(at 166.37 102.87 0)
 			(hide yes)
 			(show_name no)
@@
 		)
 		(property "Datasheet" ""
-			(at 165.1 102.87 0)
+			(at 166.37 102.87 0)
 			(hide yes)
 			(show_name no)
@@
 		)
 		(property "Description" "Power symbol creates a global label with name \"GND\" , ground"
-			(at 165.1 102.87 0)
+			(at 166.37 102.87 0)
 			(hide yes)
 			(show_name no)
@@
 			)
 		)
-		(property "Value" "AGM60P30A"
+		(property "Value" "AGM60P30AP"
 			(at 41.91 20.32 90)
 			(show_name no)
@@
 			)
 		)
-		(property "Value" "27uH"
+		(property "Value" "33uH"
 			(at 240.03 35.052 90)
 			(show_name no)
@@
 	(symbol
 		(lib_id "Device:C")
-		(at 148.59 97.79 0)
+		(at 149.86 97.79 0)
 		(unit 1)
 		(body_style 1)
@@
 		(dnp no)
 		(property "Reference" "C24"
-			(at 149.606 95.504 0)
+			(at 150.876 95.504 0)
 			(show_name no)
 			(do_not_autoplace no)
@@
 		)
 		(property "Value" "8.2pF"
-			(at 149.86 100.33 0)
+			(at 151.13 100.33 0)
 			(show_name no)
 			(do_not_autoplace no)
@@
 		)
 		(property "Footprint" "Capacitor_SMD:C_0402_1005Metric"
-			(at 149.5552 101.6 0)
+			(at 150.8252 101.6 0)
 			(hide yes)
 			(show_name no)
@@
 		)
 		(property "Datasheet" ""
-			(at 148.59 97.79 0)
+			(at 149.86 97.79 0)
 			(hide yes)
 			(show_name no)
@@
 		)
 		(property "Description" "Unpolarized capacitor"
-			(at 148.59 97.79 0)
+			(at 149.86 97.79 0)
 			(hide yes)
 			(show_name no)
@@
 	(symbol
 		(lib_id "Device:Crystal_GND24")
-		(at 157.48 92.71 0)
+		(at 158.75 92.71 0)
 		(unit 1)
 		(body_style 1)
@@
 		(dnp no)
 		(property "Reference" "Y1"
-			(at 165.608 85.344 0)
+			(at 166.878 85.344 0)
 			(show_name no)
 			(do_not_autoplace no)
@@
 		)
 		(property "Value" "X322516MLB4SI"
-			(at 165.608 87.884 0)
+			(at 166.878 87.884 0)
 			(show_name no)
 			(do_not_autoplace no)
@@
 		)
 		(property "Footprint" "Crystal:Crystal_SMD_3225-4Pin_3.2x2.5mm"
-			(at 157.48 92.71 0)
+			(at 158.75 92.71 0)
 			(hide yes)
 			(show_name no)
@@
 		)
 		(property "Datasheet" ""
-			(at 157.48 92.71 0)
+			(at 158.75 92.71 0)
 			(hide yes)
 			(show_name no)
@@
 		)
 		(property "Description" "Four pin crystal, GND on pins 2 and 4"
-			(at 157.48 92.71 0)
+			(at 158.75 92.71 0)
 			(hide yes)
 			(show_name no)
@@
 	(symbol
 		(lib_id "power:GND")
-		(at 148.59 102.87 0)
+		(at 149.86 102.87 0)
 		(unit 1)
 		(body_style 1)
@@
 		(dnp no)
 		(property "Reference" "#PWR048"
-			(at 148.59 109.22 0)
+			(at 149.86 109.22 0)
 			(hide yes)
 			(show_name no)
@@
 		)
 		(property "Value" "GND"
-			(at 148.59 106.68 0)
+			(at 149.86 106.68 0)
 			(show_name no)
 			(do_not_autoplace no)
@@
 		)
 		(property "Footprint" ""
-			(at 148.59 102.87 0)
+			(at 149.86 102.87 0)
 			(hide yes)
 			(show_name no)
@@
 		)
 		(property "Datasheet" ""
-			(at 148.59 102.87 0)
+			(at 149.86 102.87 0)
 			(hide yes)
 			(show_name no)
@@
 		)
 		(property "Description" "Power symbol creates a global label with name \"GND\" , ground"
-			(at 148.59 102.87 0)
+			(at 149.86 102.87 0)
 			(hide yes)
 			(show_name no)
